File: omnikeyish_pcb/keyboard.sch (KiCad schematic (older format))
At the start: 344 parts, among them SW1.1 KEY_P11, SW1.10 KEY_F6, SW1.11 KEY_F7, SW1.12 KEY_F8, SW1.13 KEY_F9, SW1.14 KEY_F10, SW1.15 KEY_F11, SW1.16 KEY_F12, SW1.17 KEY_PRINTSCREEN, SW1.18 KEY_SCROLL_LOCK, SW1.19 KEY_PAUSE, SW1.2 KEY_P12, SW1.20 KEY_VOLMUTE, SW1.21 KEY_VOLDOWN, SW1.22 KEY_VOLUP, SW1.23 KEY_POWER, SW1.3 KEY_ESCAPE, SW1.5 KEY_F1, SW1.6 KEY_F2, SW1.7 KEY_F3, SW1.8 KEY_F4, SW1.9 KEY_F5, SW1B.1 KEY_P11, SW1B.10 KEY_F6, SW1B.11 KEY_F7, SW1B.12 KEY_F8, SW1B.13 KEY_F9, SW1B.14 KEY_F10, SW1B.15 KEY_F11, SW1B.16 KEY_F12, SW1B.17 KEY_PRINTSCREEN, SW1B.18 KEY_SCROLL_LOCK, SW1B.19 KEY_PAUSE, SW1B.2 KEY_P12, SW1B.3 KEY_ESCAPE, SW1B.5 KEY_F1, SW1B.6 KEY_F2, SW1B.7 KEY_F3, SW1B.8 KEY_F4, SW1B.9 KEY_F5, SW1C.1 KEY_P11, SW1C.2 KEY_P12, SW1D.1 KEY_P11, SW1D.2 KEY_P12, SW2.1 KEY_P1, SW2.10 KEY_7, SW2.11 KEY_8, SW2.12 KEY_9, SW2.13 KEY_0, SW2.14 KEY_MINUS, SW2.15 KEY_EQUALS, SW2.16 KEY_BACKSPACE, SW2.17 KEY_INSERT, SW2.18 KEY_HOME, SW2.19 KEY_PGUP, SW2.2 KEY_P2, SW2.20 KEY_NUMLOCK, SW2.21 KEY_NUMDIVIDE, SW2.22 KEY_NUMTIMES, SW2.23 KEY_NUMMINUS, SW2.3 KEY_BACKQUOTE, SW2.4 KEY_1, SW2.5 KEY_2, SW2.6 KEY_3, SW2.7 KEY_4, SW2.8 KEY_5, SW2.9 KEY_6, SW2B.1 KEY_P1, SW2B.17 KEY_BIGINSERT, SW2B.2 KEY_P2, SW2C.1 KEY_P1, SW2C.2 KEY_P2, SW3.1 KEY_P3, SW3.10 KEY_U, SW3.11 KEY_I, SW3.12 KEY_O, SW3.13 KEY_P, SW3.14 KEY_LEFTBRACKET, SW3.15 KEY_RIGHTBRACKET, SW3.16 KEY_ANSIBACKSLASH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

Commit message: Rev 1.2: Fix brainfart matrix postion for Ultra's 1.5u insert and delete keys was wrong
Parts:
- removed SW2B.17: KEY_BIGINSERT, MX_Alps_Hybrid:MX-1.5U-NoLED, symbol Switch:SW_Push
- removed SW3B.17: KEY_BIGDELETE, MX_Alps_Hybrid:MX-1.5U-NoLED, symbol Switch:SW_Push
- added SW6B.17: KEY_ULTRAINSERT, MX_Alps_Hybrid:MX-1.5U-NoLED, symbol Switch:SW_Push
- added SW6B.19: KEY_ULTRADELETE, MX_Alps_Hybrid:MX-1.5U-NoLED, symbol Switch:SW_Push
Connections:
- net ROW6: now also SW6B.17.2, SW6B.19.2
- net at D6.17.2 (A), SW6.17.2: now also SW6B.17.1
- net at D6.19.2 (A), SW6.19.2: now also SW6B.19.1
Changed lines of the file:
@@
 	0    -1   -1   0
 $EndComp
-Connection ~ 19900 6450
-Wire Wire Line
-	19900 6550 19900 6450
 $Comp
 L Switch:SW_Push SW6B.16
@@
 	18850 11000 18950 11000
 Connection ~ 18850 10400
-$Comp
-L Switch:SW_Push SW3B.17
-U 1 1 5CE184EF
-P 19950 7700
-F 0 "SW3B.17" V 20125 7750 50  0000 L CNN
-F 1 "KEY_BIGDELETE" V 19775 7725 50  0000 L CNN
-F 2 "MX_Alps_Hybrid:MX-1.5U-NoLED" H 19950 7900 50  0001 C CNN
-F 3 "" H 19950 7900 50  0001 C CNN
-	1    19950 7700
-	0    -1   -1   0
-$EndComp
-Connection ~ 19950 7400
-Wire Wire Line
-	19950 7400 19950 7500
-Wire Wire Line
-	19950 7900 19950 8000
-Wire Wire Line
-	19950 8000 20050 8000
 Wire Wire Line
 	18850 8850 18850 8950
@@
 	0    -1   -1   0
 $EndComp
-Wire Wire Line
-	19900 6950 19900 7050
-$Comp
-L Switch:SW_Push SW2B.17
-U 1 1 5CBB5F1A
-P 19900 6750
-F 0 "SW2B.17" V 19700 6825 50  0000 L CNN
-F 1 "KEY_BIGINSERT" V 20100 6875 50  0000 L CNN
-F 2 "MX_Alps_Hybrid:MX-1.5U-NoLED" H 19900 6950 50  0001 C CNN
-F 3 "" H 19900 6950 50  0001 C CNN
-	1    19900 6750
-	0    -1   -1   0
-$EndComp
 Text GLabel 6400 4650 1    50   Input ~ 0
 COL3
@@
 Wire Wire Line
 	18950 8000 19050 8000
-Wire Wire Line
-	18950 7400 19950 7400
 Connection ~ 18950 7400
 Wire Wire Line
@@
 Wire Wire Line
 	20050 8000 20050 7900
-Wire Wire Line
-	19950 7400 20050 7400
 Connection ~ 20050 7400
 Wire Wire Line
 	20050 7500 20050 7400
-Connection ~ 20050 8000
 Wire Wire Line
 	20050 8000 20150 8000
@@
 	-1   0    0    1
 $EndComp
-$Comp
-L Switch:SW_Push SW6.19
-U 1 1 5D151851
-P 22400 10700
-F 0 "SW6.19" V 22354 10848 50  0000 L CNN
-F 1 "KEY_RIGHT" V 22445 10848 50  0000 L CNN
-F 2 "MX_Alps_Hybrid:MX-1U-NoLED" H 22400 10900 50  0001 C CNN
-F 3 "" H 22400 10900 50  0001 C CNN
-	1    22400 10700
-	0    1    1    0
-$EndComp
 Connection ~ 22400 10400
 Wire Wire Line
@@
 	18950 10500 18950 10400
 Wire Wire Line
-	18950 10400 20050 10400
+	18950 10400 19925 10400
 Connection ~ 20050 10400
 Wire Wire Line
 	20050 10500 20050 10400
 Wire Wire Line
-	21250 10400 22400 10400
+	21250 10400 22275 10400
 Wire Wire Line
 	20050 10400 21250 10400
@@
 $EndComp
 Wire Wire Line
-	19900 6450 20050 6450
-Wire Wire Line
 	20050 6450 21250 6450
 Connection ~ 20050 6450
@@
 	20050 6550 20050 6450
 Wire Wire Line
-	19900 7050 20050 7050
-Wire Wire Line
 	20050 7050 20150 7050
-Connection ~ 20050 7050
 Wire Wire Line
 	20050 7050 20050 6950
@@
 	0    1    1    0
 $EndComp
-Wire Wire Line
-	18950 6450 19900 6450
 Connection ~ 18950 6450
 Wire Wire Line
@@
 $EndComp
 Wire Wire Line
-	4875 12225 5350 12225
-Wire Wire Line
 	4100 14475 4100 14000
 Connection ~ 4100 14475
@@
 	3600 8000 3700 8000
 NoConn ~ 4250 16625
+Wire Wire Line
+	18950 6450 20050 6450
+Wire Wire Line
+	18950 7400 20050 7400
+$Comp
+L Switch:SW_Push SW6B.17
+U 1 1 5E80B38D
+P 19925 10700
+F 0 "SW6B.17" V 20050 10825 50  0000 L CNN
+F 1 "KEY_ULTRAINSERT" V 19525 10575 50  0000 L CNN
+F 2 "MX_Alps_Hybrid:MX-1.5U-NoLED" H 19925 10900 50  0001 C CNN
+F 3 "" H 19925 10900 50  0001 C CNN
+	1    19925 10700
+	0    -1   -1   0
+$EndComp
+$Comp
+L Switch:SW_Push SW6.19
+U 1 1 5D151851
+P 22400 10700
+F 0 "SW6.19" V 22354 10848 50  0000 L CNN
+F 1 "KEY_RIGHT" V 22445 10848 50  0000 L CNN
+F 2 "MX_Alps_Hybrid:MX-1U-NoLED" H 22400 10900 50  0001 C CNN
+F 3 "" H 22400 10900 50  0001 C CNN
+	1    22400 10700
+	0    1    1    0
+$EndComp
+$Comp
+L Switch:SW_Push SW6B.19
+U 1 1 5E980504
+P 22275 10700
+F 0 "SW6B.19" V 22450 10775 50  0000 L CNN
+F 1 "KEY_ULTRADELETE" V 22075 10750 50  0000 L CNN
+F 2 "MX_Alps_Hybrid:MX-1.5U-NoLED" H 22275 10900 50  0001 C CNN
+F 3 "" H 22275 10900 50  0001 C CNN
+	1    22275 10700
+	0    -1   -1   0
+$EndComp
+Wire Wire Line
+	22275 10500 22275 10400
+Connection ~ 22275 10400
+Wire Wire Line
+	22275 10400 22400 10400
+Wire Wire Line
+	22275 10900 22275 11000
+Wire Wire Line
+	22275 11000 22400 11000
+Connection ~ 22400 11000
+Wire Wire Line
+	19925 10500 19925 10400
+Connection ~ 19925 10400
+Wire Wire Line
+	19925 10400 20050 10400
+Wire Wire Line
+	19925 10900 19925 11000
+Wire Wire Line
+	19925 11000 20050 11000
+Connection ~ 20050 11000
 $EndSCHEMATC
