File: at101_pcb/keyboard.sch (KiCad schematic (older format))
At the start: 17 parts, among them U1 Teensy2.0

Commit message: Correct AT10[12]W? switch labels
Parts:
- renumbered D2 to D1, D1 to D2, R2 to R1, R3 to R2, R1 to R3
Changed lines of the file:
@@
 $EndComp
 $Comp
-L Device:R R3
+L Device:R R2
 U 1 1 5E839E73
 P 3425 1800
-F 0 "R3" H 3300 1650 50  0000 L CNN
+F 0 "R2" H 3300 1650 50  0000 L CNN
 F 1 "330Ω" V 3425 1700 50  0000 L CNN
 F 2 "Resistor_THT:R_Axial_DIN0207_L6.3mm_D2.5mm_P10.16mm_Horizontal" V 3355 1800 50  0001 C CNN
@@
 $EndComp
 $Comp
-L Device:R R1
+L Device:R R3
 U 1 1 5E8454AF
 P 1875 1625
-F 0 "R1" H 1925 1625 50  0000 L CNN
+F 0 "R3" H 1925 1625 50  0000 L CNN
 F 1 "330Ω" V 1875 1525 50  0000 L CNN
 F 2 "Resistor_THT:R_Axial_DIN0207_L6.3mm_D2.5mm_P10.16mm_Horizontal" V 1805 1625 50  0001 C CNN
@@
 $EndComp
 $Comp
-L Device:LED D2
+L Device:LED D1
 U 1 1 5E85229C
 P 1550 2925
-F 0 "D2" V 1650 3075 50  0000 R CNN
+F 0 "D1" V 1650 3075 50  0000 R CNN
 F 1 "NUM_LOCK_LED" V 1550 3600 50  0000 R CNN
 F 2 "LED_THT:LED_Rectangular_W5.0mm_H2.0mm" H 1550 2925 50  0001 C CNN
@@
 $EndComp
 $Comp
-L Device:LED D1
+L Device:LED D2
 U 1 1 5E8557A4
 P 3425 2775
-F 0 "D1" V 3525 2875 50  0000 R CNN
+F 0 "D2" V 3525 2875 50  0000 R CNN
 F 1 "CAPS_LOCK_LED" V 3375 3475 50  0000 R CNN
 F 2 "LED_THT:LED_Rectangular_W5.0mm_H2.0mm" H 3425 2775 50  0001 C CNN
@@
 $EndComp
 $Comp
-L Device:R R2
+L Device:R R1
 U 1 1 5E845B42
 P 1550 1800
-F 0 "R2" H 1425 1650 50  0000 L CNN
+F 0 "R1" H 1425 1650 50  0000 L CNN
 F 1 "330Ω" V 1550 1700 50  0000 L CNN
 F 2 "Resistor_THT:R_Axial_DIN0207_L6.3mm_D2.5mm_P10.16mm_Horizontal" V 1480 1800 50  0001 C CNN
